File: compass-pcb/compass-xiao-pcb/_autosave-compass-xiao-pcb.kicad_pcb (KiCad board)
At the start: 2 copper layers, 186.5 x 72.9 mm, 45 parts

Commit message: removing large board
Parts:
- moved 10K 8.60 mm to (204.6, 88.9), turned to 90 degrees
- moved QMC5883L 4.35 mm to (196.6, 94.7), turned to 90 degrees
Connections:
- QMC5883L pad 2: GND -> (no net)
Routing:
- net (no net): track 2059.0 -> 2049.0 mm
